File: hardware/kicad/accessbridge.kicad_pcb (KiCad board)
At the start: 2 copper layers, 86 x 56 mm, 64 parts, among them J1 PWR+RELAY, J2 BELL+DPS, J3 Qwiic, J4 OUT, J5 EXP, Q1 AO3400A, SW1 PAIR, U1 AP63205WU-7, U2 XIAO_ESP32C6, U3 EL357N(C)(TA)-G, U4 EL357N(C)(TA)-G, U5 EL357N(C)(TA)-G, U6 CPC1014NTR

Commit message: HW-1.1 Rev B: USB-C power input; 3D-printable enclosure (DIN + wall)
- J6 power-only USB-C (5.1k CC, 500 mA PTC, SMAJ5.0A), diode-OR into the
  XIAO 5V pin and a new V_LOOP rail for the contact loops
- Board widened to 96 x 56 mm; Rev A placement and routing kept,
  incremental update/lock workflow in gen_pcb.py
- Regenerated fabrication data (HW-1.1 Rev B ZIP, BOM, CPL, renders, STEP)
- Parametric CadQuery enclosure: DIN-rail base, wall-screw base, lid,
  PAIR plunger, cable clamp; fit check against the PCB STEP; CI job
- Docs, tests plan and changelog updated

Co-Authored-By: Claude Opus 5.5 <noreply@anthropic.com>
Claude-Session: https://claude.ai/code/session_017ugbcLJnibWHxuv1cA2VcH
Parts:
- added C11: 10u/25V, Capacitor_SMD:C_0805_2012Metric, F.Cu at (131.0, 78.0)
- added D13: SS14, Diode_SMD:D_SMA, F.Cu at (126.0, 62.0)
- added D14: SMAJ5.0A, Diode_SMD:D_SMA, F.Cu at (131.0, 58.0)
- added D15: SS14, Diode_SMD:D_SMA, F.Cu at (126.0, 74.0)
- added D16: SS14, Diode_SMD:D_SMA, F.Cu at (131.0, 70.0)
- added F2: 500mA/30V, Fuse:Fuse_1206_3216Metric, F.Cu at (126.0, 55.0)
- added J6: USB-C 5V, Connector_USB:USB_C_Receptacle_GCT_USB4125-xx-x_6P_TopMnt_Horizontal, F.Cu at (123.0, 43.4)
- added R22: 5.1k, Resistor_SMD:R_0603_1608Metric, F.Cu at (123.0, 49.6)
- added R23: 5.1k, Resistor_SMD:R_0603_1608Metric, F.Cu at (126.5, 49.6)
- moved H2 10.0 mm to (132.0, 44.0)
- moved H4 10.0 mm to (132.0, 92.0)
Connections:
- R10 pad 1: +12V -> /V_LOOP
- R14 pad 1: +12V -> /V_LOOP
- R18 pad 1: +12V -> /V_LOOP
Routing:
- net /V_LOOP: track 0.00 -> 110.9 mm, vias 0 -> 4
- net GND: track 349.7 -> 393.4 mm
- net /VBUS_F: track 0.00 -> 37.1 mm
- net /+5V_XIAO: track 49.7 -> 67.3 mm, vias 1 -> 3
- net /VBUS: track 0.00 -> 15.2 mm
- net /CC2: track 0.00 -> 6.43 mm, vias 0 -> 2
- net +3V3: track 132.1 -> 127.0 mm, vias 2 -> 4
- net /CC1: track 0.00 -> 4.46 mm
- net +12V: track 125.2 -> 127.6 mm, vias 3 -> 1
- net /IN1_A: track 12.6 -> 10.9 mm
Other:
- board size 86 x 56 mm -> 96 x 56 mm
- board text added: "AccessBridge C6 HW-1.1 Rev B"
- board text added: "AccessBridge C6 HW-1.1 Rev B - CERN-OHL-S-2.0"
- board text added: "Board 96 x 56 mm, 1.6 mm FR-4, 2 layers, 1 mm corner radius"
- board text added: "J6 USB-C: 5V power only (no data)"
- board text added: "Supply: UA-Hub LINE 12V or USB-C 5V - no mains"
- board text added: "USB 5V"
- board text removed: "AccessBridge C6 HW-1.0 Rev A"
- board text removed: "AccessBridge C6 HW-1.0 Rev A - CERN-OHL-S-2.0"
- board text removed: "Board 86 x 56 mm, 1.6 mm FR-4, 2 layers, 1 mm corner radius"
- board text removed: "Supply: UA-Hub LINE 12V DC only - no mains"

Commit message: Doorbell: any-source blueprint, no-neutral wiring options; wetting-current jumpers
- doorbell-notify blueprint accepts the AccessBridge counter, an event entity
  (e.g. Shelly input) or a binary sensor (e.g. battery Zigbee contact sensor);
  restore/reconnect ignored, optional event-type filter; 3 new tests (15/15)
- wiring.md: doorbell routes for 230 V bells without neutral at the push
  (coupling relay at the bell + battery Zigbee sensor, or cable to J2);
  Shelly 1L/2L and Eltako ER61-UC limitations documented
- Rev B (not manufactured): JP3-JP5 + R24-R26 (1k 1206, C4410) select ~3.3 or
  ~6 mA loop current per input; incremental routing, ERC/DRC clean incl. parity
- Regenerated fabrication data, renders, PCB STEP; enclosure fit check passes

Co-Authored-By: Claude Opus 5.5 <noreply@anthropic.com>
Claude-Session: https://claude.ai/code/session_017ugbcLJnibWHxuv1cA2VcH
Parts:
- added JP3: SolderJumper_2_Open, Jumper:SolderJumper-2_P1.3mm_Open_RoundedPad1.0x1.5mm, F.Cu at (49.2, 64.5)
- added JP4: SolderJumper_2_Open, Jumper:SolderJumper-2_P1.3mm_Open_RoundedPad1.0x1.5mm, F.Cu at (61.6, 62.0)
- added JP5: SolderJumper_2_Open, Jumper:SolderJumper-2_P1.3mm_Open_RoundedPad1.0x1.5mm, F.Cu at (77.6, 62.0)
- added R24: 1k, Resistor_SMD:R_1206_3216Metric, F.Cu at (52.0, 64.5)
- added R25: 1k, Resistor_SMD:R_1206_3216Metric, F.Cu at (64.4, 62.0)
- added R26: 1k, Resistor_SMD:R_1206_3216Metric, F.Cu at (80.4, 62.0)
Routing:
- net /IN1_A: track 10.9 -> 18.8 mm
- net /IN3_A: track 10.9 -> 17.8 mm
- net /IN2_A: track 11.0 -> 17.5 mm
- net +12V: track 127.6 -> 133.5 mm
- net GND: track 393.4 -> 398.3 mm
- net /IN3_WET: track 0.00 -> 3.68 mm
- net /IN2_WET: track 0.00 -> 3.68 mm
- net /IN1_WET: track 0.00 -> 3.68 mm
- net /V_LOOP: track 110.9 -> 107.6 mm, vias 4 -> 5
- net +3V3: track 127.0 -> 125.5 mm, vias 4 -> 3
- net /IN1_SIG: track 59.3 -> 60.2 mm

Commit message: BOM: optocouplers U3-U5 = UMW EL357C (C725794); sync footprint values on update
Co-Authored-By: Claude Opus 5.5 <noreply@anthropic.com>
Claude-Session: https://claude.ai/code/session_017ugbcLJnibWHxuv1cA2VcH
Parts:
- U3, U4, U5: value EL357N(C)(TA)-G -> EL357C
Changed lines of the file:
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@@
 			)
 		)
-		(property "Value" "EL357N(C)(TA)-G"
+		(property "Value" "EL357C"
 			(at 0 2.8 0)
 			(layer "F.Fab")
@@
 			)
 		)
-		(property "LCSC" "C29981"
+		(property "LCSC" "C725794"
 			(at 0 0 0)
 			(layer "F.Fab")
@@
 			)
 		)
-		(property "MPN" "EL357N(C)(TA)-G"
+		(property "MPN" "EL357C"
 			(at 0 0 0)
 			(layer "F.Fab")
@@
 			)
 		)
-		(property "Manufacturer" "Everlight"
+		(property "Manufacturer" "UMW"
 			(at 0 0 0)
 			(layer "F.Fab")
@@
 			)
 		)
-		(property "Value" "EL357N(C)(TA)-G"
+		(property "Value" "EL357C"
 			(at 0 2.8 0)
 			(layer "F.Fab")
@@
 			)
 		)
-		(property "LCSC" "C29981"
+		(property "LCSC" "C725794"
 			(at 0 0 0)
 			(layer "F.Fab")
@@
 			)
 		)
-		(property "MPN" "EL357N(C)(TA)-G"
+		(property "MPN" "EL357C"
 			(at 0 0 0)
 			(layer "F.Fab")
@@
 			)
 		)
-		(property "Manufacturer" "Everlight"
+		(property "Manufacturer" "UMW"
 			(at 0 0 0)
 			(layer "F.Fab")
@@
 			)
 		)
-		(property "MPN" "0603 470R 1% thick film"
+		(property "MPN" "0603WAF4700T5E"
 			(at 0 0 0)
 			(layer "F.Fab")
@@
 			)
 		)
-		(property "Manufacturer" "generic"
+		(property "Manufacturer" "UNI-ROYAL"
 			(at 0 0 0)
 			(layer "F.Fab")
@@
 			)
 		)
-		(property "Value" "EL357N(C)(TA)-G"
+		(property "Value" "EL357C"
 			(at 0 2.8 0)
 			(layer "F.Fab")
@@
 			)
 		)
-		(property "LCSC" "C29981"
+		(property "LCSC" "C725794"
 			(at 0 0 0)
 			(layer "F.Fab")
@@
 			)
 		)
-		(property "MPN" "EL357N(C)(TA)-G"
+		(property "MPN" "EL357C"
 			(at 0 0 0)
 			(layer "F.Fab")
@@
 			)
 		)
-		(property "Manufacturer" "Everlight"
+		(property "Manufacturer" "UMW"
 			(at 0 0 0)
 			(layer "F.Fab")
@@
 		(layer "Dwgs.User")
 		(pts
-			(xy 40 40) (xy 40 96)
+			(xy 40 40) (xy 136 40)
 		)
-		(height 6)
+		(height -6)
 		(format
 			(prefix "")
@@
 			(keep_text_aligned yes)
 		)
-		(gr_text "56.00 mm"
-			(at 32.875 68 90)
+		(gr_text "96.00 mm"
+			(at 88 32.875 0)
 			(layer "Dwgs.User")
 			(effects
@@
 		(layer "Dwgs.User")
 		(pts
-			(xy 40 40) (xy 136 40)
+			(xy 40 40) (xy 108 40)
 		)
-		(height -6)
+		(height -12)
 		(format
 			(prefix "")
@@
 			(keep_text_aligned yes)
 		)
-		(gr_text "96.00 mm"
-			(at 88 32.875 0)
+		(gr_text "68.00 mm"
+			(at 74 26.875 0)
 			(layer "Dwgs.User")
 			(effects
@@
 		(layer "Dwgs.User")
 		(pts
-			(xy 40 40) (xy 108 40)
+			(xy 40 40) (xy 40 96)
 		)
-		(height -12)
+		(height 6)
 		(format
 			(prefix "")
@@
 			(keep_text_aligned yes)
 		)
-		(gr_text "68.00 mm"
-			(at 74 26.875 0)
+		(gr_text "56.00 mm"
+			(at 32.875 68 90)
 			(layer "Dwgs.User")
 			(effects
@@
 		(net_name "")
 		(layers "F.Cu" "B.Cu")
-		(name "Antenna keep-out")
+		(name "Antenna end: no pour")
 		(hatch edge 0.5)
 		(connect_pads
@@
 		(filled_areas_thickness no)
 		(keepout
-			(tracks not_allowed)
-			(vias not_allowed)
+			(tracks allowed)
+			(vias allowed)
 			(pads allowed)
 			(copperpour not_allowed)
@@
 		(polygon
 			(pts
-				(xy 98.8 64) (xy 117.2 64) (xy 117.2 73) (xy 98.8 73)
+				(xy 98.8 59) (xy 117.2 59) (xy 117.2 64) (xy 98.8 64)
 			)
 		)
@@
 		(net_name "")
 		(layers "F.Cu" "B.Cu")
-		(name "Antenna end: no pour")
+		(name "Antenna keep-out")
 		(hatch edge 0.5)
 		(connect_pads
@@
 		(filled_areas_thickness no)
 		(keepout
-			(tracks allowed)
-			(vias allowed)
+			(tracks not_allowed)
+			(vias not_allowed)
 			(pads allowed)
 			(copperpour not_allowed)
@@
 		(polygon
 			(pts
-				(xy 98.8 59) (xy 117.2 59) (xy 117.2 64) (xy 98.8 64)
+				(xy 98.8 64) (xy 117.2 64) (xy 117.2 73) (xy 98.8 73)
 			)
 		)

Commit message: BOM: D4 PWR LED = KT-0603YG yellow-green (C2289), green 0603 out of stock
Co-Authored-By: Claude Opus 5.5 <noreply@anthropic.com>
Claude-Session: https://claude.ai/code/session_017ugbcLJnibWHxuv1cA2VcH
Parts:
- D4: value green -> yellow-green
Changed lines of the file:
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@@
 			)
 		)
-		(property "Value" "green"
+		(property "Value" "yellow-green"
 			(at 0 1.43 180)
 			(layer "F.Fab")
@@
 			)
 		)
-		(property "LCSC" "C72043"
+		(property "LCSC" "C2289"
 			(at 0 0 0)
 			(layer "F.Fab")
@@
 			)
 		)
-		(property "MPN" "KT-0603G (emerald)"
+		(property "MPN" "KT-0603YG"
 			(at 0 0 0)
 			(layer "F.Fab")
@@
 		(layer "Dwgs.User")
 		(pts
-			(xy 40 40) (xy 136 40)
+			(xy 132 44) (xy 132 92)
 		)
-		(height -6)
+		(height -8)
 		(format
 			(prefix "")
@@
 			(keep_text_aligned yes)
 		)
-		(gr_text "96.00 mm"
-			(at 88 32.875 0)
+		(gr_text "48.00 mm"
+			(at 138.875 68 90)
 			(layer "Dwgs.User")
 			(effects
@@
 		(layer "Dwgs.User")
 		(pts
-			(xy 132 44) (xy 132 92)
+			(xy 40 40) (xy 136 40)
 		)
-		(height -8)
+		(height -6)
 		(format
 			(prefix "")
@@
 			(keep_text_aligned yes)
 		)
-		(gr_text "48.00 mm"
-			(at 138.875 68 90)
+		(gr_text "96.00 mm"
+			(at 88 32.875 0)
 			(layer "Dwgs.User")
 			(effects
@@
 		(layer "Dwgs.User")
 		(pts
-			(xy 44 92) (xy 132 92)
+			(xy 40 40) (xy 40 96)
 		)
-		(height 8)
+		(height 6)
 		(format
 			(prefix "")
@@
 			(keep_text_aligned yes)
 		)
-		(gr_text "88.00 mm"
-			(at 88 98.875 0)
+		(gr_text "56.00 mm"
+			(at 32.875 68 90)
 			(layer "Dwgs.User")
 			(effects
@@
 		(layer "Dwgs.User")
 		(pts
-			(xy 40 40) (xy 108 40)
+			(xy 44 92) (xy 132 92)
 		)
-		(height -12)
+		(height 8)
 		(format
 			(prefix "")
@@
 			(keep_text_aligned yes)
 		)
-		(gr_text "68.00 mm"
-			(at 74 26.875 0)
+		(gr_text "88.00 mm"
+			(at 88 98.875 0)
 			(layer "Dwgs.User")
 			(effects
@@
 		(layer "Dwgs.User")
 		(pts
-			(xy 40 40) (xy 40 96)
+			(xy 40 40) (xy 108 40)
 		)
-		(height 6)
+		(height -12)
 		(format
 			(prefix "")
@@
 			(keep_text_aligned yes)
 		)
-		(gr_text "56.00 mm"
-			(at 32.875 68 90)
+		(gr_text "68.00 mm"
+			(at 74 26.875 0)
 			(layer "Dwgs.User")
 			(effects
